Commit message: Added inertia and collision to URDF model

File: bumperbot_description/urdf/bumperbot.urdf (robot description, URDF)
Before this commit: robot bumperbot, 6 links, 5 joints
Links:
- link base_link: mass None -> 8.2573504e-01; geometry collision mesh filename=package://bumperbot_description/meshes/base_link.STL; visual mesh filename=package://bumperbot_description/meshes/base_link.STL
- link caster_front_link: mass None -> 1.44379265037903E-06; geometry collision sphere radius=0.005; visual mesh filename=package://bumperbot_description/meshes/caster_front_link.STL
- link caster_rear_link: mass None -> 1.44379265037902E-06; geometry collision sphere radius=0.005; visual mesh filename=package://bumperbot_description/meshes/caster_rear_link.STL
- link wheel_left_link: mass None -> 0.0530086043217644; geometry collision sphere radius=0.033; visual mesh filename=package://bumperbot_description/meshes/wheel_left_link.STL
- link wheel_right_link: mass None -> 0.0530086090966721; geometry collision sphere radius=0.033; visual mesh filename=package://bumperbot_description/meshes/wheel_right_link.STL
